Commit message: [Enhance]: 收敛 GUI 驱动的采集辨识流程
- 增加 PySide6 工作台入口，覆盖模型加载、激励生成、采集、辨识、导出和历史运行浏览。

- 优化激励轨迹生成、MoveIt/RViz 校验预览、URDF 限位解析和 SIA 示例配置。

- 收敛采集后 manifest 自动填入、motion.csv 预览、辨识预测图加载和轨迹取消逻辑。

- 修正 dataset_recorder 字符串数组参数声明，补充 GUI、轨迹、采集和辨识回归测试。

验证：PYTHONPATH=src/robotdynid_ros2:/opt/ros/jazzy/lib/python3.12/site-packages:/home/betavion/work/acados/interfaces/acados_template QT_QPA_PLATFORM=offscreen venv/bin/python -m pytest src/robotdynid_ros2/test/test_gui_main_window.py src/robotdynid_ros2/test/test_gui_command_builder.py src/robotdynid_ros2/test/test_gui_artifact_model.py src/robotdynid_ros2/test/test_config.py src/robotdynid_ros2/test/test_identify_codegen_cli.py src/robotdynid_ros2/test/test_dataset_recorder_node.py

验证：./build.bash

File: examples/sia/sia_v3_urdf.urdf (robot description, URDF)
Before this commit: robot sia_v3_urdf, 8 links, 7 joints
Joints:
- joint joint1: limit lower=-2.5 upper=2.5 effort=10.0 velocity=5.1 -> lower=-3.141592653589793 upper=3.141592653589793 effort=8.0 velocity=5.0
- joint joint2: limit lower=-3.2 upper=3.2 effort=10.0 velocity=5.1 -> lower=-1.5707963267948966 upper=1.5707963267948966 effort=20.0 velocity=5.0
- joint joint3: limit lower=-1.6 upper=2.0 effort=10.0 velocity=5.1 -> lower=-1.5707963267948966 upper=1.5707963267948966 effort=20.0 velocity=5.0
- joint joint4: limit lower=-0.5 upper=3.2 effort=4.0 velocity=20.1 -> lower=-2.0943951023931953 upper=2.0943951023931953 effort=4.0 velocity=20.0
- joint joint5: limit lower=-3.2 upper=3.2 effort=4.0 velocity=20.1 -> lower=-1.5707963267948966 upper=1.5707963267948966 effort=4.0 velocity=20.0
- joint joint6: limit lower=-6.3 upper=1.0 effort=4.0 velocity=20.1 -> lower=-6.283185307179586 upper=6.283185307179586 effort=4.0 velocity=20.0
