Commit message: [Fix]: 同步 SIA 三段杆长运动学参数
- 将 link1、link4 轴向长度各增加 0.5 mm
- 将 link6 轴向长度增加 2 mm

验证：check_urdf examples/sia/sia_v3_urdf.urdf

File: examples/sia/sia_v3_urdf.urdf (robot description, URDF)
Before this commit: robot sia_v3_urdf, 8 links, 7 joints
Joints:
- joint joint1: origin xyz=0 0 0.1596 rpy=0 0 0 -> xyz=0 0 0.1601 rpy=0 0 0
- joint joint4: origin xyz=0.071 -0.351 0 rpy=1.5708 -1.5708 0 -> xyz=0.071 -0.3515 0 rpy=1.5708 -1.5708 0
- joint joint_tool: origin xyz=0 0 0.0664999999999999 rpy=0 0 0 -> xyz=0 0 0.0685 rpy=0 0 0
